File: led_panel/led_panel.kicad_pcb (KiCad board)
At the start: 4 copper layers, 330 x 330 mm, 331 parts, among them J101 19V 5A Molex, J301 DEBUG_OUT, U201 MP8759GD, U202 IND_SMALL, U301 WS2812B, U302 WS2812B, U303 WS2812B, U304 WS2812B, U305 WS2812B, U306 WS2812B, U307 WS2812B, U308 WS2812B, U309 WS2812B, U310 WS2812B, U311 WS2812B, U312 WS2812B, U313 WS2812B, U314 WS2812B, U315 WS2812B, U316 WS2812B, U317 WS2812B, U318 WS2812B, U319 WS2812B, U320 WS2812B, U321 WS2812B, U322 WS2812B, U323 WS2812B, U324 WS2812B, U325 WS2812B, U326 WS2812B, U327 WS2812B, U328 WS2812B, U329 WS2812B, U330 WS2812B, U331 WS2812B, U332 WS2812B, U333 WS2812B, U334 WS2812B, U335 WS2812B, U336 WS2812B, U337 WS2812B, U338 WS2812B, U339 WS2812B, U340 WS2812B, U341 WS2812B, U342 WS2812B, U343 WS2812B, U344 WS2812B, U345 WS2812B, U346 WS2812B, U347 WS2812B, U348 WS2812B, U349 WS2812B, U350 WS2812B, U351 WS2812B, U352 WS2812B, U353 WS2812B, U354 WS2812B, U355 WS2812B, U356 WS2812B, U357 WS2812B, U358 WS2812B, U359 WS2812B, U360 WS2812B, U361 WS2812B, U362 WS2812B, U363 WS2812B, U364 WS2812B, U365 WS2812B, U366 WS2812B, U367 WS2812B, U368 WS2812B, U369 WS2812B, U370 WS2812B, U371 WS2812B, U372 WS2812B, U373 WS2812B, U374 WS2812B, U375 WS2812B, U376 WS2812B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

Commit message: placing led
Parts:
- moved U201 605.4 mm to (-175.5, 376.1), turned to 0 degrees
- moved U557 605.4 mm to (-129.5, 377.2), turned to 0 degrees
- moved U202 602.2 mm to (-168.0, 376.1), turned to 0 degrees
- moved U558 602.2 mm to (-122.0, 377.2), turned to 0 degrees
- moved R101 364.4 mm to (529.2, 284.5)
- moved J3001 321.4 mm to (530.9, 345.4)
- moved U3225 264.1 mm to (181.9, 268.5)
- moved U3218 258.6 mm to (189.4, 261.0)
- moved U3242 256.9 mm to (189.4, 283.5)
- moved U3209 241.9 mm to (181.9, 253.5)
- moved U3236 237.6 mm to (204.4, 276.0)
- moved U3253 232.4 mm to (211.9, 291.0)
- moved U3227 231.9 mm to (196.9, 268.5)
- moved U3177 226.7 mm to (181.9, 223.5)
- moved U3205 223.5 mm to (211.9, 246.0)
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- renumbered J301 to J3001, U421 to U3001, U413 to U3002, U405 to U3003, U397 to U3004, U389 to U3005, U381 to U3006, U373 to U3007, U365 to U3008, U357 to U3009, U349 to U3010, U341 to U3011, U333 to U3012, U325 to U3013, U317 to U3014, U309 to U3015, U301 to U3016, U422 to U3017, U414 to U3018, U406 to U3019, U398 to U3020, U390 to U3021, U382 to U3022, U374 to U3023, U366 to U3024, U358 to U3025, U350 to U3026, U342 to U3027, U334 to U3028, U326 to U3029, U318 to U3030, U310 to U3031, U302 to U3032, U423 to U3033, U415 to U3034, U407 to U3035, U399 to U3036, U391 to U3037, U383 to U3038, U375 to U3039, U367 to U3040, U359 to U3041, U351 to U3042, U343 to U3043, U335 to U3044, U327 to U3045, U319 to U3046, U311 to U3047, U303 to U3048, U424 to U3049, U416 to U3050, U408 to U3051, U400 to U3052, U392 to U3053, U384 to U3054, U376 to U3055, U368 to U3056, U360 to U3057, U352 to U3058, U344 to U3059, U336 to U3060, U328 to U3061, U320 to U3062, U312 to U3063, U304 to U3064, U425 to U3065, U417 to U3066, U409 to U3067, U401 to U3068, U393 to U3069, U385 to U3070, U377 to U3071, U369 to U3072, U361 to U3073, U353 to U3074, U345 to U3075, U337 to U3076, U329 to U3077, U321 to U3078, U313 to U3079, U305 to U3080, U426 to U3081, U418 to U3082, U410 to U3083, U402 to U3084, U394 to U3085, U386 to U3086, U378 to U3087, U370 to U3088, U362 to U3089, U354 to U3090, U346 to U3091, U338 to U3092, U330 to U3093, U322 to U3094, U314 to U3095, U306 to U3096, U427 to U3097, U419 to U3098, U411 to U3099, U403 to U3100, U395 to U3101, U387 to U3102, U379 to U3103, U371 to U3104, U363 to U3105, U355 to U3106, U347 to U3107, U339 to U3108, U331 to U3109, U323 to U3110, U315 to U3111, U307 to U3112, U428 to U3113, U420 to U3114, U412 to U3115, U404 to U3116, U396 to U3117, U388 to U3118, U380 to U3119, U372 to U3120, U364 to U3121, U356 to U3122, U348 to U3123, U340 to U3124, U332 to U3125, U324 to U3126, U316 to U3127, U308 to U3128, U429 to U3129, U430 to U3130, U431 to U3131, U432 to U3132, U433 to U3133, U434 to U3134, U435 to U3135, U436 to U3136, U437 to U3137, U438 to U3138, U439 to U3139, U440 to U3140, U441 to U3141, U442 to U3142, U443 to U3143, U444 to U3144, U445 to U3145, U446 to U3146, U447 to U3147, U448 to U3148, U449 to U3149, U450 to U3150, U451 to U3151, U452 to U3152, U453 to U3153, U454 to U3154, U455 to U3155, U456 to U3156, U457 to U3157, U458 to U3158, U459 to U3159, U460 to U3160, U461 to U3161, U462 to U3162, U463 to U3163, U464 to U3164, U465 to U3165, U466 to U3166, U467 to U3167, U468 to U3168, U469 to U3169, U470 to U3170, U471 to U3171, U472 to U3172, U473 to U3173, U474 to U3174, U475 to U3175, U476 to U3176, U477 to U3177, U478 to U3178, U479 to U3179, U480 to U3180, U481 to U3181, U482 to U3182, U483 to U3183, U484 to U3184, U485 to U3185, U486 to U3186, U487 to U3187, U488 to U3188, U489 to U3189, U490 to U3190, U491 to U3191, U492 to U3192, U493 to U3193, U494 to U3194, U495 to U3195, U496 to U3196, U497 to U3197, U498 to U3198, U499 to U3199, U500 to U3200, U501 to U3201, U502 to U3202, U503 to U3203, U504 to U3204, U505 to U3205, U506 to U3206, U507 to U3207, U508 to U3208, U509 to U3209, U510 to U3210, U511 to U3211, U512 to U3212, U513 to U3213, U514 to U3214, U515 to U3215, U516 to U3216, U517 to U3217, U518 to U3218, U519 to U3219, U520 to U3220, U521 to U3221, U522 to U3222, U523 to U3223, U524 to U3224, U525 to U3225, U526 to U3226, U527 to U3227, U528 to U3228, U529 to U3229, U530 to U3230, U531 to U3231, U532 to U3232, U533 to U3233, U534 to U3234, U535 to U3235, U536 to U3236, U537 to U3237, U538 to U3238, U539 to U3239, U540 to U3240, U541 to U3241, U542 to U3242, U543 to U3243, U544 to U3244, U545 to U3245, U546 to U3246, U547 to U3247, U548 to U3248, U549 to U3249, U550 to U3250, U551 to U3251, U552 to U3252, U553 to U3253, U554 to U3254, U555 to U3255, U556 to U3256
Connections:
- U201 pad 6: Net-(U201-Pad6) -> Net-(R212-Pad2)
- U201 pad 9: Net-(U201-Pad9) -> Net-(C219-Pad2)
